File: PCB/PCB.kicad_sch (KiCad schematic)
At the start: 125 parts, among them SW1 SW_Push, SW10 SW_Push, SW11 SW_Push, SW12 SW_Push, SW13 SW_Push, SW14 SW_Push, SW15 SW_Push, SW16 SW_Push, SW17 SW_Push, SW18 SW_Push, SW19 SW_Push, SW2 SW_Push, SW20 SW_Push, SW21 SW_Push, SW22 SW_Push, SW23 SW_Push, SW24 SW_Push, SW25 SW_Push, SW26 SW_Push, SW27 SW_Push, SW28 SW_Push, SW29 SW_Push, SW3 SW_Push, SW30 SW_Push, SW31 SW_Push, SW32 SW_Push, SW33 SW_Push, SW34 SW_Push, SW35 SW_Push, SW36 SW_Push, SW37 SW_Push, SW38 SW_Push, SW39 SW_Push, SW4 SW_Push, SW40 SW_Push, SW41 SW_Push, SW42 SW_Push, SW43 SW_Push, SW44 SW_Push, SW45 SW_Push, SW46 SW_Push, SW47 SW_Push, SW48 SW_Push, SW49 SW_Push, SW5 SW_Push, SW50 SW_Push, SW51 SW_Push, SW52 SW_Push, SW53 SW_Push, SW54 SW_Push, SW55 SW_Push, SW56 SW_Push, SW57 SW_Push, SW58 SW_Push, SW59 SW_Push, SW6 SW_Push, SW60 SW_Push, SW61 SW_Push, SW62 SW_Push, SW7 SW_Push, SW8 SW_Push, SW9 SW_Push

Commit message: Added PCB
Parts:
- D1, D10, D11, D12, D13, D14, D15, D16, D17, D18, D19, D2, D20, D21, D22, D23, D24, D25, D26, D27, D28, D29, D3, D30, D31, D32, D33, D34, D35, D36, D37, D38, D39, D4, D40, D41, D42, D43, D44, D45, D46, D47, D48, D49, D5, D50, D51, D52, D53, D54, D55, D56, D57, D58, D59, D6, D60, D61, D62, D7, D8, D9: footprint (none) -> Diode_THT:D_DO-35_SOD27_P7.62mm_Horizontal
- SW1, SW10, SW11, SW12, SW13, SW14, SW15, SW16, SW17, SW18, SW19, SW2, SW20, SW21, SW22, SW23, SW24, SW25, SW26, SW27, SW28, SW3, SW30, SW31, SW32, SW33, SW34, SW35, SW36, SW37, SW38, SW39, SW4, SW40, SW43, SW44, SW45, SW46, SW47, SW48, SW49, SW5, SW50, SW51, SW52, SW54, SW55, SW56, SW58, SW59, SW6, SW60, SW61, SW62, SW7, SW8, SW9: footprint (none) -> Button_Switch_Keyboard:SW_Cherry_MX_1.00u_PCB
- SW29, SW41: footprint (none) -> Button_Switch_Keyboard:SW_Cherry_MX_2.00u_PCB
- SW42, SW53: footprint (none) -> Button_Switch_Keyboard:SW_Cherry_MX_2.25u_PCB
- SW57: footprint (none) -> Button_Switch_Keyboard:SW_Cherry_MX_6.25u_PCB
Connections:
- net COL11: no longer SW54.1
- net COL13: now also SW54.1
Other:
- moved on the sheet: D54, SW54

Commit message: Ready to SHip!
Parts:
- removed D62: D, Diode_THT:D_DO-35_SOD27_P7.62mm_Horizontal, symbol Device:D
- removed SW62: SW_Push, Button_Switch_Keyboard:SW_Cherry_MX_1.00u_PCB, symbol Switch:SW_Push
- SW29, SW41: footprint Button_Switch_Keyboard:SW_Cherry_MX_2.00u_PCB -> Button_Switch_Keyboard:SW_Cherry_MX_1.00u_PCB
- SW42, SW53: footprint Button_Switch_Keyboard:SW_Cherry_MX_2.25u_PCB -> Button_Switch_Keyboard:SW_Cherry_MX_1.00u_PCB
- SW57: footprint Button_Switch_Keyboard:SW_Cherry_MX_6.25u_PCB -> Button_Switch_Keyboard:SW_Cherry_MX_1.00u_PCB
Connections:
- net COL0: now also SW42.1, SW54.1; no longer SW43.1, SW55.1
- net COL1: now also SW43.1, SW55.1; no longer SW44.1, SW56.1
- net COL10: now also SW52.1, SW59.1; no longer SW53.1
- net COL11: now also SW53.1
- net COL12: now also SW61.1
- net COL13: no longer SW42.1, SW54.1
- net COL2: now also SW44.1, SW56.1; no longer SW45.1, SW57.1
- net COL3: now also SW45.1; no longer SW46.1, SW58.1
- net COL4: now also SW46.1, SW57.1; no longer SW47.1, SW59.1
- net COL5: now also SW47.1; no longer SW48.1, SW60.1
- net COL6: now also SW48.1; no longer SW49.1, SW61.1
- net COL7: now also SW49.1; no longer SW50.1
- net COL8: now also SW50.1; no longer SW51.1
- net COL9: now also SW51.1, SW58.1; no longer SW52.1
- net ROW2: no longer D42.1 (K)
- net ROW3: now also D42.1 (K); no longer D54.1 (K)
- net ROW4: now also D54.1 (K)
- net at D60.2 (A): now also SW60.1; no longer SW60.2
