File: PCB/PCB.kicad_pcb (KiCad board)
At the start: 2 copper layers, 302.8 x 133.1 mm, 125 parts, among them SW1 SW_Push, SW10 SW_Push, SW11 SW_Push, SW12 SW_Push, SW13 SW_Push, SW14 SW_Push, SW15 SW_Push, SW16 SW_Push, SW17 SW_Push, SW18 SW_Push, SW19 SW_Push, SW2 SW_Push, SW20 SW_Push, SW21 SW_Push, SW22 SW_Push, SW23 SW_Push, SW24 SW_Push, SW25 SW_Push, SW26 SW_Push, SW27 SW_Push, SW28 SW_Push, SW29 SW_Push, SW3 SW_Push, SW30 SW_Push, SW31 SW_Push, SW32 SW_Push, SW33 SW_Push, SW34 SW_Push, SW35 SW_Push, SW36 SW_Push, SW37 SW_Push, SW38 SW_Push, SW39 SW_Push, SW4 SW_Push, SW40 SW_Push, SW41 SW_Push, SW42 SW_Push, SW43 SW_Push, SW44 SW_Push, SW45 SW_Push, SW46 SW_Push, SW47 SW_Push, SW48 SW_Push, SW49 SW_Push, SW5 SW_Push, SW50 SW_Push, SW51 SW_Push, SW52 SW_Push, SW53 SW_Push, SW54 SW_Push, SW55 SW_Push, SW56 SW_Push, SW57 SW_Push, SW58 SW_Push, SW59 SW_Push, SW6 SW_Push, SW60 SW_Push, SW61 SW_Push, SW62 SW_Push, SW7 SW_Push, SW8 SW_Push, SW9 SW_Push

Commit message: Ready to SHip!
Parts:
- removed D62: D, Diode_THT:D_DO-35_SOD27_P7.62mm_Horizontal
- removed SW62: SW_Push, Button_Switch_Keyboard:SW_Cherry_MX_1.00u_PCB
- SW29, SW41: footprint Button_Switch_Keyboard:SW_Cherry_MX_2.00u_PCB -> Button_Switch_Keyboard:SW_Cherry_MX_1.00u_PCB
- SW42, SW53: footprint Button_Switch_Keyboard:SW_Cherry_MX_2.25u_PCB -> Button_Switch_Keyboard:SW_Cherry_MX_1.00u_PCB
- SW57: footprint Button_Switch_Keyboard:SW_Cherry_MX_6.25u_PCB -> Button_Switch_Keyboard:SW_Cherry_MX_1.00u_PCB
- moved A1 50.5 mm to (48.4, 66.8), turned to 0 degrees
- moved D42 42.8 mm to (92.6, 116.6)
- moved D29 37.5 mm to (87.8, 97.5)
- moved D30 37.5 mm to (114.0, 97.5)
- moved D31 37.5 mm to (133.1, 97.5)
- moved D32 37.5 mm to (152.1, 97.5)
- moved D33 37.5 mm to (171.2, 97.5)
- moved D34 37.5 mm to (190.2, 97.5)
- moved D35 37.5 mm to (209.3, 97.5)
- moved D36 37.5 mm to (228.3, 97.5)
- moved D37 37.5 mm to (247.4, 97.5)
- moved D38 37.5 mm to (266.4, 97.5)
- moved D41 37.5 mm to (335.5, 97.5)
- moved SW29 37.5 mm to (82.8, 94.5)
- moved SW30 37.5 mm to (109.0, 94.5)
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Connections:
- D42 pad 1: ROW2 -> ROW3
- D54 pad 1: ROW3 -> ROW4
- SW42 pad 1: COL13 -> COL0
- SW43 pad 1: COL0 -> COL1
- SW44 pad 1: COL1 -> COL2
- SW45 pad 1: COL2 -> COL3
- SW46 pad 1: COL3 -> COL4
- SW47 pad 1: COL4 -> COL5
- SW48 pad 1: COL5 -> COL6
- SW49 pad 1: COL6 -> COL7
- SW50 pad 1: COL7 -> COL8
- SW51 pad 1: COL8 -> COL9
- SW52 pad 1: COL9 -> COL10
- SW53 pad 1: COL10 -> COL11
- SW54 pad 1: COL13 -> COL0
- SW55 pad 1: COL0 -> COL1
- SW56 pad 1: COL1 -> COL2
- SW57 pad 1: COL2 -> COL4
- SW58 pad 1: COL3 -> COL9
- SW59 pad 1: COL4 -> COL10
- SW60 pad 1: COL5 -> Net-(D60-A)
- SW60 pad 2: Net-(D60-A) -> unconnected-(SW60-Pad2)
- SW61 pad 1: COL6 -> COL12
Routing:
- net COL13: track 542.7 -> 326.7 mm, vias 1 -> 3
- net COL7: track 440.3 -> 248.8 mm, vias 12 -> 0
- net ROW4: track 540.2 -> 400.5 mm, vias 9 -> 0
- net COL5: track 295.9 -> 192.4 mm, vias 2 -> 9
- net ROW0: track 518.8 -> 430.0 mm, vias 17 -> 4
- net COL3: track 246.4 -> 166.5 mm
- net ROW3: track 499.1 -> 426.1 mm, vias 15 -> 3
- net COL12: track 298.0 -> 367.7 mm, vias 3 -> 4
- net COL6: track 306.1 -> 247.5 mm, vias 0 -> 5
- net COL0: track 189.2 -> 134.9 mm, vias 3 -> 0
- net COL4: track 263.6 -> 217.7 mm, vias 2 -> 4
- net COL11: track 288.7 -> 329.7 mm, vias 3 -> 2
- net ROW1: track 516.7 -> 479.3 mm, vias 19 -> 3
- net COL10: track 360.4 -> 332.2 mm, vias 1 -> 2
- net COL9: track 276.7 -> 304.0 mm, vias 8 -> 2
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Other:
- board size 302.8 x 133.1 mm -> 317.6 x 110.4 mm
- board text added: "Made By Richit"
- board text added: "Richit"
- board text removed: "Richit's Keyboard"

Commit message: Ship time maybe
Parts:
- SW1, SW10, SW11, SW12, SW13, SW14, SW15, SW16, SW17, SW18, SW19, SW2, SW20, SW21, SW22, SW23, SW24, SW25, SW26, SW27, SW28, SW29, SW3, SW30, SW31, SW32, SW33, SW34, SW35, SW36, SW37, SW38, SW39, SW4, SW40, SW41, SW42, SW43, SW44, SW45, SW46, SW47, SW48, SW49, SW5, SW50, SW51, SW52, SW53, SW54, SW55, SW56, SW57, SW58, SW59, SW6, SW60, SW61, SW7, SW8, SW9: footprint Button_Switch_Keyboard:SW_Cherry_MX_1.00u_PCB -> Richit:SW_Cherry_MX_1.00u_PCB_MOD
